File: Add-On_Boards/LiBo_BaseBoard/LiBo_BaseBoard/LiBo_BaseBoard.kicad_pcb (KiCad board)
At the start: 2 copper layers, 28 parts, among them IC2 ADS1015IDGSR, IC3 DAC7311IDCKR, J1 USB_C_Receptacle_USB2.0, J2 2199230-3, J3 KH-BNC50-3511, J4 KH-BNC50-3511, J5 Conn_01x16, U1 USBLC6-2SC6, U2 TLV62568DBV

Commit message: Finish Schem - Begin Layout
Parts:
- removed IC3: DAC7311IDCKR, Github_Library:SOT65P210X110-6N
- added C10: 10u, Capacitor_SMD:C_0805_2012Metric_Pad1.18x1.45mm_HandSolder, F.Cu at (220.2, 30.1)
- added C11: 100n, Capacitor_SMD:C_0805_2012Metric_Pad1.18x1.45mm_HandSolder, F.Cu at (220.2, 27.9)
- added C12: 100n, Capacitor_SMD:C_0805_2012Metric_Pad1.18x1.45mm_HandSolder, F.Cu at (139.8, 101.8)
- added C13: 10u, Capacitor_SMD:C_0805_2012Metric_Pad1.18x1.45mm_HandSolder, F.Cu at (141.9, 101.8)
- added C8: 100n, Capacitor_SMD:C_0805_2012Metric_Pad1.18x1.45mm_HandSolder, F.Cu at (221.4, 63.0)
- added C9: 4u7, Capacitor_SMD:C_0805_2012Metric_Pad1.18x1.45mm_HandSolder, F.Cu at (174.1, 95.3)
- added D1: LED, LED_SMD:LED_0805_2012Metric_Pad1.15x1.40mm_HandSolder, F.Cu at (147.1, 30.7)
- added D2: LED, LED_SMD:LED_0805_2012Metric_Pad1.15x1.40mm_HandSolder, F.Cu at (147.3, 36.0)
- added D3: LED, LED_SMD:LED_0805_2012Metric_Pad1.15x1.40mm_HandSolder, F.Cu at (147.4, 40.8)
- added IC1: MCP1702T-5002E_MB, Github_Library:MCP1703T5002EMB, F.Cu at (113.7, 74.1)
- added IC4: SN74LVC125APWR, Github_Library:SN74LVC125APWR, F.Cu at (226.0, 69.3)
- added J10: Conn_01x18, Connector_PinHeader_2.54mm:PinHeader_1x18_P2.54mm_Horizontal, F.Cu at (213.1, 123.9)
- added J6: TF_PUSH, Github_Library:TFPUSH, F.Cu at (242.5, 69.0)
- added J7: Conn_ST_STDC14, Connector_PinHeader_1.27mm:PinHeader_2x07_P1.27mm_Vertical, F.Cu at (263.1, 61.8)
- added J8: Conn_01x10, Connector_PinHeader_2.54mm:PinHeader_1x10_P2.54mm_Vertical, F.Cu at (153.3, 93.1)
- added LED1: WS2812C-2020, Github_Library:WS2812C2020, F.Cu at (144.2, 61.9)
- added R10: 3k3, Resistor_SMD:R_0805_2012Metric_Pad1.20x1.40mm_HandSolder, F.Cu at (227.2, 76.7)
- added R11: 3k3, Resistor_SMD:R_0805_2012Metric_Pad1.20x1.40mm_HandSolder, F.Cu at (229.4, 63.0)
- added R12: 3k3, Resistor_SMD:R_0805_2012Metric_Pad1.20x1.40mm_HandSolder, F.Cu at (220.3, 69.0)
- added R13: 10k, Resistor_SMD:R_0805_2012Metric_Pad1.20x1.40mm_HandSolder, F.Cu at (170.2, 46.2)
- added R14: 10k, Resistor_SMD:R_0805_2012Metric_Pad1.20x1.40mm_HandSolder, F.Cu at (166.9, 46.2)
- added R15: 10k, Resistor_SMD:R_0805_2012Metric_Pad1.20x1.40mm_HandSolder, F.Cu at (202.9, 118.1)
- added R16: 3k3, Resistor_SMD:R_0805_2012Metric_Pad1.20x1.40mm_HandSolder, F.Cu at (128.7, 101.7)
- added R17: 3k3, Resistor_SMD:R_0805_2012Metric_Pad1.20x1.40mm_HandSolder, F.Cu at (213.5, 23.7)
- added R18: 10k, Resistor_SMD:R_0805_2012Metric_Pad1.20x1.40mm_HandSolder, F.Cu at (210.5, 118.2)
- added R19: 5k1, Resistor_SMD:R_0805_2012Metric_Pad1.20x1.40mm_HandSolder, F.Cu at (147.1, 32.8)
- added R20: 5k1, Resistor_SMD:R_0805_2012Metric_Pad1.20x1.40mm_HandSolder, F.Cu at (147.3, 38.0)
- added R21: 5k1, Resistor_SMD:R_0805_2012Metric_Pad1.20x1.40mm_HandSolder, F.Cu at (147.4, 42.9)
- added R9: 3k3, Resistor_SMD:R_0805_2012Metric_Pad1.20x1.40mm_HandSolder, F.Cu at (224.2, 76.7)
- added U3: MCP4725A0T-E/CH, Package_TO_SOT_SMD:SOT-23-6, F.Cu at (220.2, 24.8)
- L1: footprint Inductor_SMD_Wurth:L_Wurth_WE-LQSH-4020 -> LED_SMD:LED_0805_2012Metric_Pad1.15x1.40mm_HandSolder
- moved J4 167.0 mm to (225.2, 109.7), turned to -90 degrees
- moved J3 125.2 mm to (225.2, 89.6), turned to -90 degrees
- moved R3 97.8 mm to (208.8, 48.7), turned to -90 degrees
- moved R8 94.6 mm to (208.4, 95.2), turned to -90 degrees
- moved U1 94.0 mm to (202.1, 54.4)
- moved RV1 92.3 mm to (165.4, 93.3), turned to 90 degrees
- moved J1 86.8 mm to (202.2, 45.8), turned to 180 degrees
- moved R2 85.0 mm to (195.6, 48.7), turned to -90 degrees
- moved J5 57.3 mm to (172.8, 99.0)
- moved R4 52.6 mm to (88.9, 79.1), turned to -90 degrees
- moved L1 46.8 mm to (96.5, 74.1)
- moved J2 43.6 mm to (177.8, 70.0), turned to -90 degrees
- moved U2 43.2 mm to (95.6, 79.1), turned to 180 degrees
- moved C7 42.6 mm to (144.6, 65.0)
- moved C4 28.4 mm to (91.0, 79.2), turned to -90 degrees
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Connections:
- IC2 pad 1: unconnected-(IC2-ADDR-Pad1) -> Earth
- IC2 pad 10: unconnected-(IC2-SCL-Pad10) -> /GPIO36
- IC2 pad 2: unconnected-(IC2-ALERT/RDY-Pad2) -> /ADC_RDY
- IC2 pad 3: unconnected-(IC2-GND-Pad3) -> Earth
- IC2 pad 4: unconnected-(IC2-AIN0-Pad4) -> /ADC_HDR_IN0
- IC2 pad 5: unconnected-(IC2-AIN1-Pad5) -> /ADC_BNC_IN1
- IC2 pad 6: unconnected-(IC2-AIN2-Pad6) -> /ADC_HDR_IN2
- IC2 pad 7: unconnected-(IC2-AIN3-Pad7) -> /ADC_HDR_IN3
- IC2 pad 8: unconnected-(IC2-VDD-Pad8) -> +3V3
- IC2 pad 9: unconnected-(IC2-SDA-Pad9) -> /GPIO35
- J2 pad 24: /GPIO18 -> /DAC_MCU_OUT
- J2 pad 34: /GPIO33 -> /ADC_RDY
- J2 pad 35: /GPIO12 -> /CS0_SPI
- J2 pad 36: /GPIO34 -> /ADC_MCU_IN0
- J2 pad 52: /MTCK -> /JTAG_MTCK
- J2 pad 54: /MTDO -> /JTAG_MTDO
- J2 pad 58: /MTDI -> /JTAG_MTDI
- J2 pad 60: /MTMS -> /JTAG_MTMS
- J2 pad 64: /U0TXD -> /JTAG_VCP_RX
- J2 pad 66: /U0RXD -> /JTAG_VCP_TX
- J3 pad 1: unconnected-(J3-Pad1) -> Earth
- J3 pad 2: unconnected-(J3-Pad2) -> /DAC_BNC_OUT
- J4 pad 1: unconnected-(J4-Pad1) -> Earth
- J4 pad 2: unconnected-(J4-Pad2) -> /ADC_BNC_IN1
Routing:
- net /GPIO3: track 31.4 -> 0.00 mm
- net +3V3: track 0.00 -> 24.2 mm, vias 0 -> 3
- net /DO_SDCARD: track 0.00 -> 17.7 mm
- net /GPIO11: track 0.00 -> 17.2 mm
- net Earth: track 0.00 -> 12.6 mm, vias 0 -> 9
- net /USB_D+: track 0.00 -> 12.5 mm
- net /GPIO13: track 0.00 -> 11.7 mm
- net /DI_SDCARD: track 0.00 -> 11.6 mm
- net /USB_D-: track 0.00 -> 11.3 mm
- net /GPIO14: track 0.00 -> 10.1 mm
- net Net-(U2-EN): track 0.00 -> 9.71 mm, vias 0 -> 2
- net /SCK_SDCARD: track 0.00 -> 9.16 mm
- net /CS_SDCARD: track 0.00 -> 7.97 mm
- net /USB_CC1: track 0.00 -> 7.72 mm
- net Net-(IC4-3A): track 0.00 -> 7.62 mm
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Other:
- board text added: "1 2 3 4"
- board text added: "3V3"
- board text added: "5V"
- board text added: "ADC"
- board text added: "BOOT"
- board text added: "DAC"
- board text added: "I2C P/U"
- board text added: "JTAG"
- board text added: "LED"
- board text added: "MicroSD"
- board text added: "RST"
- board text added: "USB"
- board text added: "VBUS"
- board text added: "VBUS->3V3"
- board text added: "VBUS->5V"

Commit message: Added stuff
Parts:
- C1, C10, C11, C12, C13, C2, C4, C5, IC1, IC2, L1, R16, R17, R4, R5, R6, U2, U3: moved to B.Cu
- moved J7 111.3 mm to (152.1, 70.7)
- moved R4 108.6 mm to (191.9, 44.8)
- moved C2 108.5 mm to (214.2, 46.5)
- moved C4 104.6 mm to (189.8, 44.8)
- moved IC1 100.6 mm to (210.1, 45.1)
- moved U2 96.1 mm to (185.3, 44.8), turned to 0 degrees
- moved R5 95.5 mm to (185.0, 51.1), turned to 0 degrees
- moved R6 95.5 mm to (185.0, 48.7), turned to 180 degrees
- moved U3 95.0 mm to (179.0, 110.4), turned to -90 degrees
- moved L1 94.2 mm to (184.3, 39.8), turned to 180 degrees
- moved R7 93.6 mm to (165.8, 47.5)
- moved C11 90.9 mm to (182.1, 110.4), turned to -90 degrees
- moved C6 90.6 mm to (163.7, 47.5), turned to -90 degrees
- moved C1 90.4 mm to (204.7, 46.5)
- moved C10 88.0 mm to (184.3, 110.4), turned to -90 degrees
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Connections:
- J8 pad 4: /GPIO37 -> /JTAG_MTMS
- J8 pad 7: /JTAG_MTMS -> /JTAG_MTCK
- J8 pad 8: /JTAG_MTCK -> /GPIO38
- J8 pad 9: /GPIO38 -> /GPIO37
Routing:
- net /JTAG_VCP_RX: track 0.00 -> 64.6 mm, vias 0 -> 3
- net /JTAG_VCP_TX: track 0.00 -> 64.1 mm, vias 0 -> 1
- net /JTAG_MTMS: track 0.00 -> 60.8 mm, vias 0 -> 3
- net /GPIO37: track 0.00 -> 59.0 mm, vias 0 -> 1
- net /JTAG_MTDI: track 0.00 -> 57.0 mm, vias 0 -> 1
- net /JTAG_MTDO: track 0.00 -> 54.9 mm, vias 0 -> 1
- net /GPIO38: track 0.00 -> 53.6 mm, vias 0 -> 3
- net /JTAG_MTCK: track 0.00 -> 52.4 mm, vias 0 -> 1
- net +5V: track 0.00 -> 47.8 mm, vias 0 -> 1
- net VBUS: track 6.65 -> 23.2 mm, vias 1 -> 2
- net Earth: track 12.6 -> 22.1 mm, vias 9 -> 17
- net +3V3: track 24.2 -> 31.4 mm, vias 3 -> 4
Other:
- board outline added: 98.9 x 96.6 mm
- board text added: "5V 3V3 GND MISO MOSI CS0 SCK GND SDA SCL GND ADC_3 ADC_2 ADC_1 ADC_0 GND DAC GND"
- board text added: "GND 5V V0 RS R/W E D0 D1 D2 D3 D4 D5 D6 D7 A K"
- board text removed: "1 2 3 4"
