File: Add-On_Boards/LiBo_BaseBoard/LiBo_BaseBoard/LiBo_BaseBoard.kicad_pcb (KiCad board)
At the start: 2 copper layers, 92.4 x 96.6 mm, 63 parts, among them IC1 MCP1702T-5002E_MB, IC2 ADS1015IDGSR, IC4 SN74LVC125APWR, J1 USB_C_Receptacle_USB2.0, J10 Conn_01x18, J2 2199230-3, J3 KH-BNC50-3511, J4 KH-BNC50-3511, J5 Conn_01x16, J6 TF_PUSH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

Commit message: Almost finished layout - BaseBoard
Parts:
- R17: moved to F.Cu
- moved R17 30.4 mm to (210.5, 106.1)
- moved J4 22.0 mm to (221.8, 87.6)
- moved J3 17.1 mm to (221.8, 106.5)
- moved R15 16.6 mm to (214.2, 100.3), turned to 180 degrees
- moved C3 11.4 mm to (231.7, 75.9)
- moved RST1 11.4 mm to (236.4, 75.9)
- moved R1 11.4 mm to (229.6, 75.9)
- moved BOOT1 10.0 mm to (236.4, 66.0)
- moved C6 10.0 mm to (231.7, 66.0)
- moved R7 10.0 mm to (229.6, 66.0)
- moved R18 6.74 mm to (214.2, 107.1), turned to 0 degrees
Routing:
- net +3V3: track 31.4 -> 332.3 mm, vias 4 -> 3
- net /GPIO35: track 6.33 -> 135.2 mm, vias 0 -> 5
- net /GPIO36: track 5.43 -> 133.0 mm, vias 0 -> 5
- net /ADC_MCU_IN0: track 2.54 -> 76.7 mm, vias 0 -> 3
- net /GPIO11: track 41.6 -> 114.1 mm, vias 0 -> 3
- net /DAC_MCU_OUT: track 0.00 -> 72.2 mm, vias 0 -> 2
- net /GPIO46: track 0.00 -> 70.8 mm, vias 0 -> 2
- net /ADC_RDY: track 5.80 -> 74.7 mm, vias 0 -> 3
- net /GPIO14: track 14.5 -> 79.5 mm, vias 0 -> 1
- net /CHIP_BOOT: track 0.00 -> 64.9 mm, vias 0 -> 2
- net /CS0_SPI: track 29.5 -> 94.0 mm, vias 0 -> 1
- net /GPIO13: track 40.9 -> 104.2 mm, vias 0 -> 1
- net /CHIP_PU: track 0.00 -> 61.2 mm, vias 0 -> 2
- net /DAC_BNC_OUT: track 0.00 -> 52.4 mm, vias 0 -> 2
- net +5V: track 44.9 -> 90.1 mm, vias 1 -> 2
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- added copper zone on B.Cu, net +3V3
- added copper zone on B.Cu, net Earth
- added copper zone on B.Cu, net Net-(U2-SW)

Commit message: Baseboard done
Parts:
- removed U$2: M.2-B-KEY, M.2-Card-Footprints:M.2-B-KEY
- added G***: LOGO, LOGO, F.Cu at (232.3, 36.8)
- moved ? 46.6 mm to (169.2, 70.0)
- moved J2 35.7 mm to (209.2, 70.0)
- moved R17 4.20 mm to (214.2, 104.0), turned to 0 degrees
- moved D3 2.13 mm to (201.8, 48.0), turned to 0 degrees
- moved R21 2.03 mm to (201.8, 50.1), turned to 0 degrees
- moved R8 0.94 mm to (207.9, 84.4), turned to 0 degrees
- moved C10 0.88 mm to (187.7, 108.2)
- moved C13 0.56 mm to (197.4, 109.5)
- moved C11 0.55 mm to (184.9, 108.2)
- moved R16 0.43 mm to (211.1, 109.6)
- moved C7 0.27 mm to (231.3, 53.6)
- moved C12 0.23 mm to (200.0, 109.5)
Connections:
- ? pad 1: (no net) -> Earth
- REF** pad 1: (no net) -> Earth (x3)
Routing:
- net +3V3: track 332.3 -> 510.0 mm, vias 3 -> 5
- net /GPIO14: track 79.5 -> 160.6 mm
- net /CS0_SPI: track 94.0 -> 156.0 mm, vias 1 -> 3
- net /GPIO13: track 104.2 -> 165.4 mm, vias 1 -> 3
- net /GPIO11: track 114.1 -> 172.6 mm
- net /GPIO35: track 135.2 -> 180.4 mm, vias 5 -> 6
- net +5V: track 90.1 -> 133.3 mm, vias 2 -> 3
- net Earth: track 48.2 -> 85.8 mm, vias 31 -> 506
- net /GPIO38: track 49.4 -> 86.6 mm
- net /JTAG_MTDI: track 52.8 -> 89.6 mm
- net /JTAG_MTCK: track 48.1 -> 85.0 mm
- net /JTAG_MTDO: track 50.7 -> 87.5 mm
- net /JTAG_VCP_TX: track 59.9 -> 96.6 mm
- net /JTAG_VCP_RX: track 60.4 -> 97.0 mm
- net /JTAG_MTMS: track 56.6 -> 93.2 mm, vias 3 -> 2
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- added copper zone on F.Cu, net Earth
- added copper zone on B.Cu, net VBUS
Other:
- outline, holes or cut-outs redrawn
- board text added: "1001000"
- board text added: "1100000"
- board text added: "3V3 JRCLK NRST MTCK MTDO MTDI MTMS VCPrx VCPtx GND"
- board text added: "ADC BNC IN"
- board text added: "ADD ADC HDR"
- board text added: "ADD DAC HDR"
- board text added: "DAC BNC OUT"
- board text added: "GPIO1 LCD_RS GPIO2 LCD_E GPIO3 LCD_D0 GPIO4 LCD_D1 GPIO5 LCD_D2 GPIO6 LCD_D3 GPIO7 LCD_D4 GPIO8 LCD_D5 GPIO9 LCD_D6 GPIO10 LCD_D7 GPIO11 SCK_SPI GPIO12 CS0_SPI GPIO13 MOSI_SPI GPIO14 MISO_SPI GPIO33 ADC_RDY GPIO34 ADC_MCU_IN0 GPIO18 DAC_MCU_OUT GPIO35 SDA GPIO36 SCL GPIO37 JTAG_JRCLK GPIO38 JTAG_NRST MTCK JTAG_MTCK MTDO JTAG_MTDO MTDI JTAG_MTDI MTMS JTAG_MTMS UOTXD JTAG_VCP_RX UORXD JTAG_VCP_TX"
- board text added: "IO46"
- board text added: "LiBO M.2 BOARD"
- board text added: "LiBo BaseBoard Designed: D.Heetkamp Version: V1.0 Date: 15-7-24"
- board text added: "RV1"

Commit message: updated the Libo M.2 main board
Parts:
- added TP1: TestPoint, TestPoint:TestPoint_Pad_D1.0mm, F.Cu at (196.6, 18.8)
- added TP2: TestPoint, TestPoint:TestPoint_Pad_D1.0mm, F.Cu at (196.6, 21.8)
- added TP3: TestPoint, TestPoint:TestPoint_Pad_D1.0mm, F.Cu at (199.7, 18.8)
- added TP4: TestPoint, TestPoint:TestPoint_Pad_D1.0mm, F.Cu at (199.7, 21.8)
- added TP5: TestPoint, TestPoint:TestPoint_Pad_D1.0mm, F.Cu at (202.7, 18.8)
- added TP6: TestPoint, TestPoint:TestPoint_Pad_D1.0mm, F.Cu at (202.7, 21.8)
Connections:
- net /ADC_BNC_IN1 renamed ADC_IN1
- net /ADC_HDR_IN0 renamed ADC_IN0
- net /ADC_HDR_IN1 renamed /OUTPUTS/ADC_HDR_IN1
- net /ADC_HDR_IN2 renamed ADC_IN2
- net /ADC_HDR_IN3 renamed ADC_IN3
- net /ADC_MCU_IN0 renamed ADC_MCU_IN0
- net /ADC_RDY renamed ADC_RDY
- net /CHIP_BOOT renamed /M.2_INPUT/CHIP_BOOT
- net /CHIP_PU renamed /M.2_INPUT/CHIP_PU
- net /CS0_SPI renamed CS0_SPI
- net /CS_SDCARD renamed CS_SDCARD
- net /DAC_MCU_OUT renamed DAC_MCU_OUT
- net /DI_SDCARD renamed DI_SDCARD
- net /DO_SDCARD renamed DO_SDCARD
- net /GPIO11 renamed SCK_SPI
- net /GPIO13 renamed MOSI_SPI
- net /GPIO14 renamed MISO_SPI
- net /GPIO17 renamed /M.2_INPUT/GPIO18
- net /GPIO21 renamed /M.2_INPUT/GPIO21
- net /GPIO35 renamed SDA
- net /GPIO36 renamed SCL
- net /GPIO37 renamed JTAG_JRCLK
- net /GPIO38 renamed JTAG_NRST
- net /GPIO45 renamed /M.2_INPUT/GPIO45
- net /JTAG_MTCK renamed JTAG_MTCK
- net /JTAG_MTDI renamed JTAG_MTDI
- net /JTAG_MTDO renamed JTAG_MTDO
- net /JTAG_MTMS renamed JTAG_MTMS
- net /JTAG_VCP_RX renamed JTAG_VCP_RX
- net /JTAG_VCP_TX renamed JTAG_VCP_TX
- net /LCD_A renamed /OUTPUTS/LCD_A
- net /LCD_V0 renamed /OUTPUTS/LCD_V0
- net /SCK_SDCARD renamed SCK_SDCARD
- net /SPICLK_N renamed /M.2_INPUT/SPICLK_N
- net /SPICLK_P renamed /M.2_INPUT/SPICLK_P
- net /SPICS1 renamed /M.2_INPUT/SPICS1
- net /USB_CC1 renamed /POWER/USB_CC1
- net /USB_CC2 renamed /POWER/USB_CC2
- J1 pad A6: /USB_D+ -> USB_D+
- J1 pad A7: /USB_D- -> USB_D-
- J1 pad B6: /USB_D+ -> USB_D+
- J1 pad B7: /USB_D- -> USB_D-
- J10 pad 2: /DAC_HDR_OUT -> DAC_OUT
- J2 pad 23: /USB_D+ -> /M.2_INPUT/USB_D+
- J2 pad 25: /USB_D- -> /M.2_INPUT/USB_D-
- J2 pad 41: /GPIO10 -> LCD_D7
- J2 pad 43: /GPIO9 -> LCD_D6
- J2 pad 47: /GPIO8 -> LCD_D5
- J2 pad 49: /GPIO7 -> LCD_D4
- J2 pad 53: /GPIO6 -> LCD_D3
- J2 pad 55: /GPIO5 -> LCD_D2
- J2 pad 59: /GPIO4 -> LCD_D1
- J2 pad 61: /GPIO3 -> LCD_D0
- J2 pad 65: /GPIO2 -> LCD_E
- J2 pad 67: /GPIO1 -> LCD_RS
- J2 pad 72: /GPIO46 -> /M.2_INPUT/GPIO46
- J3 pad 2: /DAC_BNC_OUT -> DAC_OUT
- J5 pad 10: /GPIO6 -> /OUTPUTS/LCD_D3
- J5 pad 11: /GPIO7 -> /OUTPUTS/LCD_D4
- J5 pad 12: /GPIO8 -> /OUTPUTS/LCD_D5
- J5 pad 13: /GPIO9 -> /OUTPUTS/LCD_D6
- J5 pad 14: /GPIO10 -> /OUTPUTS/LCD_D7
- J5 pad 4: /GPIO1 -> /OUTPUTS/LCD_RS
- J5 pad 6: /GPIO2 -> /OUTPUTS/LCD_E
- J5 pad 7: /GPIO3 -> /OUTPUTS/LCD_D0
- J5 pad 8: /GPIO4 -> /OUTPUTS/LCD_D1
- J5 pad 9: /GPIO5 -> /OUTPUTS/LCD_D2
- LED1 pad 3: /GPIO46 -> GPIO46
- R17 pad 1: /DAC_HDR_OUT -> Net-(R17-Pad1)
- R18 pad 1: /DAC_HDR_OUT -> Net-(R17-Pad1)
- R18 pad 2: /DAC_BNC_OUT -> DAC_OUT
- U1 pad 1: /USB_D+ -> USB_D-
- U1 pad 3: /USB_D+ -> USB_D+
- U1 pad 4: /USB_D- -> USB_D+
- U1 pad 6: /USB_D- -> USB_D-
- U3 pad 1: /DAC_BNC_OUT -> DAC_OUT
Routing:
- net (no net): track 0.00 -> 639.3 mm, vias 0 -> 2
- net /USB_D+: track 59.1 -> 0.00 mm
- net /USB_D-: track 58.8 -> 0.00 mm
- net DAC_OUT: track 0.00 -> 52.4 mm
- net /DAC_BNC_OUT: track 52.4 -> 0.00 mm
- net /GPIO1: track 51.6 -> 0.00 mm
- net /GPIO46: track 49.7 -> 0.00 mm, vias 2 -> 0
- net /GPIO3: track 48.1 -> 0.00 mm
- net /GPIO2: track 47.9 -> 0.00 mm
- net /GPIO4: track 46.7 -> 0.00 mm
- net /GPIO5: track 45.7 -> 0.00 mm
- net /GPIO6: track 44.1 -> 0.00 mm
- net /GPIO7: track 43.6 -> 0.00 mm
- net /GPIO8: track 42.2 -> 0.00 mm
- net /GPIO9: track 41.2 -> 0.00 mm
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
Commit message: first release
Parts:
- removed ? (x2): , 
- removed the G*** at (232.3, 36.8)
- removed REF** (x3): MountingHole_2.2mm_M2_DIN965_Pad, MountingHole:MountingHole_2.2mm_M2_DIN965_Pad
- added G***: LOGO, LOGO, F.Cu at (220.1, 37.1)
- added G***: LOGO, LOGO, B.Cu at (176.3, 74.6)
- TP3: moved to B.Cu
- moved TP6 88.8 mm to (214.1, 109.8)
- moved TP5 79.8 mm to (214.2, 97.7)
- moved TP4 42.9 mm to (166.4, 49.0)
- moved TP3 31.6 mm to (191.9, 49.4)
- moved TP1 23.5 mm to (200.5, 41.9)
- moved TP2 20.4 mm to (193.5, 41.9)
- moved U1 0.52 mm to (197.1, 41.8), turned to -90 degrees
Connections:
- J2 pad 23: /M.2_INPUT/USB_D+ -> USB_D+
- J2 pad 25: /M.2_INPUT/USB_D- -> USB_D-
Routing:
- net (no net): track 639.3 -> 500.4 mm
- net USB_D+: track 0.00 -> 59.2 mm
- net USB_D-: track 0.00 -> 58.7 mm
- net DAC_OUT: track 52.4 -> 72.9 mm
- net VBUS: track 64.9 -> 68.6 mm
- net Net-(R17-Pad1): track 0.00 -> 3.07 mm
- net ADC_IN1: track 46.8 -> 49.9 mm
- net Net-(U2-EN): track 9.82 -> 12.4 mm
- net CS_SDCARD: track 7.97 -> 9.60 mm
- net Earth: track 85.8 -> 86.0 mm, vias 506 -> 504
Other:
- board text added: "LiBo BaseBoard Designed: D.Heetkamp Version: V1.0 Date: 08-07-25"
- board text removed: "LiBo BaseBoard Designed: D.Heetkamp Version: V1.0 Date: 15-7-24"
