File: Add-On_Boards/LiBo_BaseBoard/LiBo_BaseBoard/LiBo_BaseBoard.kicad_sch (KiCad schematic)
At the start: 44 parts, among them IC1 MCP1702T-5002E_MB, IC2 ADS1015IDGSR, IC4 SN74LVC125APWR, J1 USB_C_Receptacle_USB2.0, J2 2199230-3, J3 KH-BNC50-3511, J4 KH-BNC50-3511, J5 Conn_01x16, J6 TF_PUSH, U1 USBLC6-2SC6, U2 TLV62568DBV, U3 MCP4725A0T-E/CH

Commit message: Finish Schem - Begin Layout
Parts:
- added D1, D2, D3: LED, LED_SMD:LED_0805_2012Metric_Pad1.15x1.40mm_HandSolder, symbol Device:LED
- added J10: Conn_01x18, Connector_PinHeader_2.54mm:PinHeader_1x18_P2.54mm_Horizontal, symbol Connector_Generic:Conn_01x18
- added J7: Conn_ST_STDC14, Connector_PinHeader_1.27mm:PinHeader_2x07_P1.27mm_Vertical, symbol Connector:Conn_ST_STDC14
- added J8: Conn_01x10, Connector_PinHeader_2.54mm:PinHeader_1x10_P2.54mm_Vertical, symbol Connector_Generic:Conn_01x10
- added R15, R18: 10k, Resistor_SMD:R_0805_2012Metric_Pad1.20x1.40mm_HandSolder, symbol Device:R
- added R16, R17: 3k3, Resistor_SMD:R_0805_2012Metric_Pad1.20x1.40mm_HandSolder, symbol Device:R
- added R19, R20, R21: 5k1, Resistor_SMD:R_0805_2012Metric_Pad1.20x1.40mm_HandSolder, symbol Device:R
- IC1: footprint GitHub_Library:MCP1703T5002EMB -> Github_Library:MCP1703T5002EMB
- L1: footprint Inductor_SMD_Wurth:L_Wurth_WE-LQSH-4020 -> LED_SMD:LED_0805_2012Metric_Pad1.15x1.40mm_HandSolder
- LED1: footprint GitHub_Library:WS2812C2020 -> Github_Library:WS2812C2020
Connections:
- net ADC_IN1 is gone; now on net ADC_BNC_IN1: IC2.5 (AIN1)
- net DAC_OUT is gone; now on net DAC_BNC_OUT: U3.1 (VOUT)
- net GPIO12 is gone; now on net CS0_SPI: J2.35
- net GPIO33 is gone; now on net ADC_RDY: J2.34
- net MISO_SPI is gone; now on net GPIO14: IC4.11 (4Y)
- net MOSI_SPI is gone; now on net GPIO13: R9.1
- net SCK_SPI is gone; now on net GPIO11: R10.1
- net SCL is gone; now on net GPIO36: IC2.10 (SCL), R13.2, U3.5 (SCL)
- net SDA is gone; now on net GPIO35: IC2.9 (SDA), R14.2, U3.4 (SDA)
- net +3V3: now also J10.17 (Pin_17), J7.3 (VCC), J8.10 (Pin_10), R20.1
- net +5V: now also J10.18 (Pin_18), R19.1
- net CS0_SPI: now also J10.13 (Pin_13)
- net Earth: now also J3.1, J4.1, D1.1 (K), D2.1 (K), D3.1 (K), J10.1 (Pin_1), J10.11 (Pin_11), J10.16 (Pin_16), J10.3 (Pin_3), J10.8 (Pin_8), J7.11 (GNDDetect), J7.5 (GND), J7.7 (GND), J8.1 (Pin_1)
- net GPIO11: now also J10.12 (Pin_12)
- net GPIO13: now also J10.14 (Pin_14)
- net GPIO14: now also J10.15 (Pin_15)
- net GPIO35: now also J10.10 (Pin_10)
- net GPIO36: now also J10.9 (Pin_9)
- net GPIO37: now also J7.9 (JRCLK/NC), J8.4 (Pin_4)
- net GPIO38: now also J7.12 (~{RST}), J8.9 (Pin_9)
- net VBUS: now also R21.1
- net ADC_BNC_IN1: now reaches J4.2
- net ADC_BNC_IN1: now also R15.1
- net DAC_BNC_OUT: now reaches J3.2
- net DAC_BNC_OUT: now also R18.2
- net ADC_IN0 renamed ADC_HDR_IN0
- net ADC_HDR_IN0: now also J10.4 (Pin_4), R16.1
- net ADC_IN2 renamed ADC_HDR_IN2
- net ADC_HDR_IN2: now also J10.6 (Pin_6)
- net ADC_IN3 renamed ADC_HDR_IN3
- net ADC_HDR_IN3: now also J10.7 (Pin_7)
- net GPIO18 renamed DAC_MCU_OUT
- net DAC_MCU_OUT: now also R17.2
- net GPIO34 renamed ADC_MCU_IN0
- net ADC_MCU_IN0: now also R16.2
- net MTCK renamed JTAG_MTCK
- net JTAG_MTCK: now also J7.6 (JCLK/SWCLK), J8.8 (Pin_8)
- net MTDI renamed JTAG_MTDI
- net JTAG_MTDI: now also J7.10 (JTDI/NC), J8.5 (Pin_5)
- net MTDO renamed JTAG_MTDO
- net JTAG_MTDO: now also J7.8 (JTDO/SWO), J8.6 (Pin_6)
- net MTMS renamed JTAG_MTMS
- net JTAG_MTMS: now also J7.4 (JTMS/SWDIO), J8.7 (Pin_7)
- net U0RXD renamed JTAG_VCP_TX
- net JTAG_VCP_TX: now also J7.14 (VCP_TX), J8.2 (Pin_2)
- net U0TXD renamed JTAG_VCP_RX
- net JTAG_VCP_RX: now also J7.13 (VCP_RX), J8.3 (Pin_3)
- new net: D1.2 (A), R19.2
- new net: D3.2 (A), R21.2
- new net: D2.2 (A), R20.2
- new net ADC_HDR_IN1: J10.5 (Pin_5), R15.2
- new net DAC_HDR_OUT: J10.2 (Pin_2), R17.1, R18.1
Other:
- note added: "I2C USED"
- note added: "JTAG/SWD"
- note added: "ST-Link Config"
- note added: "USED"
- note added: "USED FOR TESTING"
- note added: "USED SPI"
- moved on the sheet: J3, J4

Commit message: Added stuff
Parts:
- BOOT1, RST1: Manufacturer Number (none) -> EVQP2P02W
Connections:
- net GPIO37: now also J8.9 (Pin_9); no longer J8.4 (Pin_4)
- net GPIO38: now also J8.8 (Pin_8); no longer J8.9 (Pin_9)
- net JTAG_MTCK: now also J8.7 (Pin_7); no longer J8.8 (Pin_8)
- net JTAG_MTMS: now also J8.4 (Pin_4); no longer J8.7 (Pin_7)
Other:
- note added: "USB 2.0 Umax = 5V Imax = 3A"
Changed lines of the file:
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@@
 	(rectangle
 		(start 19.05 16.51)
-		(end 50.8 24.13)
+		(end 57.15 27.94)
 		(stroke
 			(width 0.5)
@@
 		)
 	)
+	(text "USB 2.0\nUmax = 5V \nImax = 3A"
+		(exclude_from_sim no)
+		(at 42.418 25.908 0)
+		(effects
+			(font
+				(size 1.5 1.5)
+				(bold yes)
+			)
+			(justify left bottom)
+		)
+	)
 	(text "USED FOR TESTING"
 		(exclude_from_sim no)
@@
 	(text "USB_C\n"
 		(exclude_from_sim no)
-		(at 20.32 21.59 0)
+		(at 25.4 23.368 0)
 		(effects
 			(font
@@
 		)
 	)
-	(label "JTAG_JRCLK"
-		(at 289.56 242.57 180)
-		(fields_autoplaced yes)
-		(effects
-			(font
-				(size 1.27 1.27)
-			)
-			(justify right bottom)
-		)
-	)
 	(label "GPIO3"
 		(at 44.45 246.38 0)
@@
 		)
 	)
-	(label "JTAG_MTCK"
+	(label "JTAG_NRST"
 		(at 289.56 232.41 180)
 		(fields_autoplaced yes)
@@
 		)
 	)
-	(label "JTAG_MTDI"
-		(at 289.56 240.03 180)
-		(fields_autoplaced yes)
-		(effects
-			(font
-				(size 1.27 1.27)
-			)
-			(justify right bottom)
-		)
-	)
 	(label "DAC_MCU_OUT"
 		(at 78.74 294.64 180)
@@
 		)
 	)
+	(label "JTAG_MTDO"
+		(at 289.56 237.49 180)
+		(fields_autoplaced yes)
+		(effects
+			(font
+				(size 1.27 1.27)
+			)
+			(justify right bottom)
+		)
+	)
 	(label "GPIO4"
 		(at 44.45 248.92 0)
@@
 		)
 	)
-	(label "JTAG_NRST"
-		(at 289.56 229.87 180)
-		(fields_autoplaced yes)
-		(effects
-			(font
-				(size 1.27 1.27)
-			)
-			(justify right bottom)
-		)
-	)
 	(label "ADC_IN2"
 		(at 229.87 165.1 180)
@@
 		)
 	)
-	(label "SCK_SPI"
-		(at 331.47 234.95 180)
+	(label "JTAG_JRCLK"
+		(at 289.56 229.87 180)
 		(fields_autoplaced yes)
 		(effects
@@
 		)
 	)
-	(label "LCD_D2"
-		(at 78.74 251.46 180)
+	(label "SCK_SPI"
+		(at 331.47 234.95 180)
 		(fields_autoplaced yes)
 		(effects
@@
 		)
 	)
-	(label "CS_SDCARD"
-		(at 283.21 101.6 0)
+	(label "LCD_D2"
+		(at 78.74 251.46 180)
 		(fields_autoplaced yes)
 		(effects
@@
 				(size 1.27 1.27)
 			)
-			(justify left bottom)
+			(justify right bottom)
 		)
 	)
-	(label "JTAG_MTDO"
-		(at 289.56 237.49 180)
+	(label "CS_SDCARD"
+		(at 283.21 101.6 0)
 		(fields_autoplaced yes)
 		(effects
@@
 				(size 1.27 1.27)
 			)
-			(justify right bottom)
+			(justify left bottom)
 		)
 	)
@@
 		)
 	)
+	(label "JTAG_MTDI"
+		(at 289.56 240.03 180)
+		(fields_autoplaced yes)
+		(effects
+			(font
+				(size 1.27 1.27)
+			)
+			(justify right bottom)
+		)
+	)
 	(label "SCK_SDCARD"
 		(at 283.21 109.22 0)
@@
 		)
 	)
+	(label "JTAG_MTCK"
+		(at 289.56 234.95 180)
+		(fields_autoplaced yes)
+		(effects
+			(font
+				(size 1.27 1.27)
+			)
+			(justify right bottom)
+		)
+	)
 	(label "CS0_SPI"
 		(at 78.74 276.86 180)
@@
 		)
 	)
+	(label "JTAG_MTMS"
+		(at 289.56 242.57 180)
+		(fields_autoplaced yes)
+		(effects
+			(font
+				(size 1.27 1.27)
+			)
+			(justify right bottom)
+		)
+	)
 	(label "LCD_A"
 		(at 311.15 154.94 180)
@@
 		)
 	)
-	(label "JTAG_MTMS"
-		(at 289.56 234.95 180)
-		(fields_autoplaced yes)
-		(effects
-			(font
-				(size 1.27 1.27)
-			)
-			(justify right bottom)
-		)
-	)
 	(label "SDA"
 		(at 229.87 157.48 180)
@@
 			)
 		)
-		(property "Datasheet" "~"
+		(property "Datasheet" "https://datasheet.lcsc.com/lcsc/2004131006_PANASONIC-EVQP2P02W_C512395.pdf"
 			(at 115.57 165.1 0)
 			(effects
@@
 			)
 		)
+		(property "Manufacturer Number" "EVQP2P02W"
+			(at 120.65 165.1 90)
+			(effects
+				(font
+					(size 1.27 1.27)
+				)
+				(hide yes)
+			)
+		)
 		(pin "1"
 		)
@@
 		(on_board yes)
 		(dnp no)
-		(fields_autoplaced yes)
 		(property "Reference" "J1"
-			(at 33.02 27.94 0)
+			(at 42.418 69.85 0)
 			(effects
 				(font
@@
 		)
 		(property "Value" "USB_C_Receptacle_USB2.0"
-			(at 33.02 30.48 0)
+			(at 33.02 31.496 0)
 			(effects
 				(font
@@
 			)
 		)
-		(property "Datasheet" "~"
+		(property "Datasheet" "https://datasheet.lcsc.com/lcsc/2004131006_PANASONIC-EVQP2P02W_C512395.pdf"
 			(at 115.57 215.9 0)
 			(effects
@@
 			(effects
 				(font
+					(size 1.27 1.27)
+				)
+				(hide yes)
+			)
+		)
+		(property "Manufacturer Number" "EVQP2P02W"
+			(at 120.65 215.9 90)
+			(effects
+				(font
