File: Add-On_Boards/LiBo_BaseBoard/LiBo_BaseBoard/Power_Page.kicad_sch (KiCad schematic)
At the start: 23 parts, among them IC1 MCP1702T-5002E_MB, J1 USB_C_Receptacle_USB2.0, U1 USBLC6-2SC6, U2 TLV62568DBV

Commit message: first release
Changed lines of the file:
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@@
 	)
 	(global_label "USB_D+"
-		(shape input)
+		(shape bidirectional)
 		(at 123.19 81.28 0)
 		(fields_autoplaced yes)
@@
 	)
 	(global_label "USB_D-"
-		(shape input)
+		(shape bidirectional)
 		(at 124.46 48.26 0)
 		(fields_autoplaced yes)
