File: Add-On_Boards/LiBo_BaseBoard/LiBo_BaseBoard/LiBo_BaseBoard-backups/LiBo_BaseBoard-2024-06-04_143602/_autosave-LiBo_BaseBoard.kicad_sch (KiCad schematic)
At the start: 57 parts, among them IC1 MCP1702T-5002E_MB, IC2 ADS1015IDGSR, IC4 SN74LVC125APWR, J1 USB_C_Receptacle_USB2.0, J10 Conn_01x18, J2 2199230-3, J3 KH-BNC50-3511, J4 KH-BNC50-3511, J5 Conn_01x16, J6 TF_PUSH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

Commit message: Improved the layout
Other:
- note added: "PWR Status LED"
Changed lines of the file:
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@@
+	)
+	(rectangle
+		(start 186.69 241.3)
+		(end 218.44 246.38)
+		(stroke
+			(width 0.5)
+			(type default)
+		)
+		(fill
+			(type none)
+		)
+	)
+	(rectangle
+		(start 186.69 241.3)
+		(end 229.87 292.1)
+		(stroke
+			(width 0.5)
+			(type default)
+		)
+		(fill
+			(type none)
+		)
 	)
 	(rectangle
@@
 		)
 	)
+	(text "PWR Status LED"
+		(exclude_from_sim no)
+		(at 189.992 245.364 0)
+		(effects
+			(font
+				(size 2 2)
+				(thickness 1)
+				(bold yes)
+			)
+			(justify left bottom)
+		)
+	)
