File: Main_Boards/LiBo_M.2_ESP32S3/ESP32S3_M.2_Board/ESP32S3_M.2_Board.kicad_pcb (KiCad board)
At the start: 4 copper layers, 23 x 42 mm, 67 parts, among them J1 USB-C, J2 M.2-B-KEY, U1 USBLC6-2SC6, U2 TLV62568DBVR, U3 ESP32-S3R8, U4 W25Q16JVUXIQ, Y1 40MHz, Y2 32.768KHz

Commit message: updated the Libo M.2 main board
Parts:
- added R13: 10k, Resistor_SMD:R_0402_1005Metric_Pad0.72x0.64mm_HandSolder, F.Cu at (237.6, 103.5)
- added TP6: TestPoint, TestPoint:TestPoint_Pad_D1.0mm, F.Cu at (220.2, 107.7)
Connections:
- J2 pad MOUNTING-HOLE: unconnected-(J2-MP1-PadMOUNTING-HOLE) -> Earth
Routing:
- net Earth: track 144.0 -> 147.3 mm
- net +3V3: track 30.3 -> 31.2 mm, vias 18 -> 17
