File: Main_Boards/LiBo_M.2_ESP32S3/ESP32S3_M.2_Board/ESP32S3_M.2_Board.kicad_pcb (KiCad board)
At the start: 4 copper layers, 23 x 42 mm, 69 parts, among them J1 USB-C, J2 M.2-B-KEY, U1 USBLC6-2SC6, U2 TLV62568DBVR, U3 ESP32-S3R8, U4 W25Q16JVUXIQ, Y1 40MHz, Y2 32.768KHz

Commit message: Add new STEP and WRL files for M.2 Arduino and ESP32S3 Boards
- Added M.2 Arduino Module Board STEP file (12633 KB)
- Added ESP32S3 M.2 Board STEP file (16645 KB)
- Added WRL file for unnamed ESP32S3 M.2 Board (2692 KB)
- Created lock file for ESP32S3 M.2 Board project
Parts:
- BOOT1, RST1: footprint Button_Switch_SMD:SW_SPST_EVQP2 -> PCB_Lib_DaanHeetkamp_KiCad:SW_SPST_EVQP2
- C1, C10, C11, C13, C14, C16, C17, C18, C19, C2, C20, C21, C22, C23, C24, C25, C26, C3, C4, C5, C6, C7, C8, C9: footprint Capacitor_SMD:C_0402_1005Metric_Pad0.74x0.62mm_HandSolder -> PCB_Lib_DaanHeetkamp_KiCad:C_0402_1005Metric_Pad0.74x0.62mm_HandSolder
- C12, C15: footprint Capacitor_SMD:C_0603_1608Metric_Pad1.08x0.95mm_HandSolder -> PCB_Lib_DaanHeetkamp_KiCad:C_0603_1608Metric_Pad1.08x0.95mm_HandSolder
- D1, D2: footprint LED_SMD:LED_0402_1005Metric_Pad0.77x0.64mm_HandSolder -> PCB_Lib_DaanHeetkamp_KiCad:LED_0402_1005Metric_Pad0.77x0.64mm_HandSolder
- G***: footprint LOGO -> PCB_Lib_DaanHeetkamp_KiCad:LOGO
- J1: footprint Connector_USB:USB_C_Receptacle_GCT_USB4105-xx-A_16P_TopMnt_Horizontal -> PCB_Lib_DaanHeetkamp_KiCad:USB_C_Receptacle_GCT_USB4105-xx-A_16P_TopMnt_Horizontal
- J2: footprint M.2-Card-Footprints:M.2-B-KEY -> PCB_Lib_DaanHeetkamp_KiCad:M.2-B-KEY
- JP1, JP2, R3, R4: footprint Resistor_SMD:R_0201_0603Metric -> PCB_Lib_DaanHeetkamp_KiCad:R_0201_0603Metric
- L1: footprint Inductor_SMD_Wurth:L_Wurth_WE-LQSH-4020 -> PCB_Lib_DaanHeetkamp_KiCad:L_Wurth_WE-LQSH-4020
- L2, L3: footprint Inductor_SMD:L_0603_1608Metric_Pad1.05x0.95mm_HandSolder -> PCB_Lib_DaanHeetkamp_KiCad:L_0603_1608Metric_Pad1.05x0.95mm_HandSolder
- R1, R10, R11, R12, R13, R2, R5, R6, R7, R8, R9: footprint Resistor_SMD:R_0402_1005Metric_Pad0.72x0.64mm_HandSolder -> PCB_Lib_DaanHeetkamp_KiCad:R_0402_1005Metric_Pad0.72x0.64mm_HandSolder
- TP1, TP10, TP2, TP3, TP4, TP5, TP6, TP7, TP8, TP9: footprint TestPoint:TestPoint_Pad_D1.0mm -> PCB_Lib_DaanHeetkamp_KiCad:TestPoint_Pad_D1.0mm
- U1: footprint Package_TO_SOT_SMD:SOT-23-6 -> PCB_Lib_DaanHeetkamp_KiCad:SOT-23-6
- U2: footprint Package_TO_SOT_SMD:SOT-23-5 -> PCB_Lib_DaanHeetkamp_KiCad:SOT-23-5
- U3: footprint Package_DFN_QFN:QFN-56-1EP_7x7mm_P0.4mm_EP4x4mm -> PCB_Lib_DaanHeetkamp_KiCad:QFN-56-1EP_7x7mm_P0.4mm_EP4x4mm
- Y1: footprint Crystal:Crystal_SMD_3225-4Pin_3.2x2.5mm -> PCB_Lib_DaanHeetkamp_KiCad:Crystal_SMD_3225-4Pin_3.2x2.5mm
- Y2: footprint Crystal:Crystal_SMD_3215-2Pin_3.2x1.5mm -> PCB_Lib_DaanHeetkamp_KiCad:Crystal_SMD_3215-2Pin_3.2x1.5mm
