File: Main_Boards/LiBo_M.2_ESP32S3/ESP32S3_M.2_Board/ESP32S3_M.2_Board.kicad_sch (KiCad schematic)
At the start: 66 parts, among them J1 USB-C, J2 M.2-B-KEY, U1 USBLC6-2SC6, U2 TLV62568DBVR, U3 ESP32-S3R8, U4 W25Q16JVUXIQ, Y1 40MHz, Y2 32.768KHz

Commit message: updated the Libo M.2 main board
Parts:
- added R13: 10k, Resistor_SMD:R_0402_1005Metric_Pad0.72x0.64mm_HandSolder, symbol Device:R
- added TP6: TestPoint, TestPoint:TestPoint_Pad_D1.0mm, symbol Connector:TestPoint
Connections:
- net +3V3: now also R13.1
- net CHIP_BOOT: now also R13.2
- net Earth: now also TP6.1
Other:
- moved on the sheet: BOOT1, C26
