File: Add-On_Boards/LiBo_ArduinoBoard/M.2_Arduino_Module_Board/M.2_Arduino_Module_Board.kicad_sch (KiCad schematic)
At the start: 15 parts, among them J2 2199230-3, J3 USB_C_Receptacle_USB2.0, U1 USBLC6-2SC6, U2 TLV62568DBV

Commit message: Changes
Parts:
- J3: symbol PCB_Lib_DaanHeetkamp:USB_C_Receptacle_USB2.0 -> KiCad_Library:USB_C_Receptacle_USB2.0
Changed lines of the file:
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@@
 	)
 	(symbol
-		(lib_id "PCB_Lib_DaanHeetkamp:USB_C_Receptacle_USB2.0")
+		(lib_id "KiCad_Library:USB_C_Receptacle_USB2.0")
 		(at 33.02 53.34 0)
 		(unit 1)
@@
 			)
 		)
-		(property "Description" ""
+		(property "Description" "USB 2.0-only Type-C Receptacle connector"
 			(at 33.02 53.34 0)
 			(effects

Commit message: Changes to ArduinoBoard
Needed:
1. Diodes.
2. Status LEDS
3. Footprint checking
Parts:
- added BOOT1: SW_BOOT, Button_Switch_SMD:SW_SPST_EVQP2, symbol Switch:SW_Push
- added C1, C2: 1u, Capacitor_SMD:C_0402_1005Metric_Pad0.74x0.62mm_HandSolder, symbol Device:C
- added C3, C6: 100n, Capacitor_SMD:C_0402_1005Metric_Pad0.74x0.62mm_HandSolder, symbol Device:C
- added IC1: MCP1702T-5002E_MB, GitHub_Library:MCP1703T5002EMB, symbol GitHub_Library:MCP1702T-5002E_MB
- added R1, R7: 10k, Resistor_SMD:R_0402_1005Metric_Pad0.72x0.64mm_HandSolder, symbol Device:R
- added R8, R9: 5k1, Resistor_SMD:R_0402_1005Metric_Pad0.72x0.64mm_HandSolder, symbol Device:R
- added RST1: SW_RST, Button_Switch_SMD:SW_SPST_EVQP2, symbol Switch:SW_Push
- A1: footprint PCB_Lib_DaanHeetkamp_KiCad:Arduino_Uno_Footprint -> GitHub_Library:Arduino_Uno_Footprint; symbol PCB_Lib_DaanHeetkamp_KiCad:Arduino_Uno_Footprint -> GitHub_Library:Arduino_Uno_Footprint; Height (none) -> 4.2; Manufacturer_Name (none) -> TE Connectivity; Manufacturer_Part_Number (none) -> 2199230-3; RS Part Number (none) -> 2175445; RS Price/Stock (none) -> http://uk.rs-online.com/web/p/products/2175445
- J2: footprint SamacSys_Parts:21992303 -> GitHub_Library:21992303; symbol SamacSys_Parts:2199230-3 -> GitHub_Library:M.2_67Con_Fem_2199230-3
- LED1: footprint PCB_Lib_DaanHeetkamp_KiCad:WS2812C2020 -> GitHub_Library:WS2812C2020; symbol PCB_Lib_DaanHeetkamp_KiCad:WS2812C-2020 -> GitHub_Library:WS2812C-2020
- renumbered C6 to C7, J3 to J1, R4 to R2, R5 to R3, R6 to R4, R7 to R5, R8 to R6
Connections:
- net +3V3: now also A1.2 (IOREF), A1.30 (AREF), A1.4 (3V3), R1.1, R7.1, R8.1, R9.1
- net CHIP_BOOT: now also BOOT1.2, C6.1, R7.2
- net CHIP_PU: now also A1.3 (~{RESET}), C3.1, R1.2, RST1.2
- net Earth: now also A1.29 (GND), A1.6 (GND), A1.7 (GND), BOOT1.1, C1.2, C2.2, C3.2, C6.2, IC1.1 (GND), RST1.1
- net GPIO1: now also A1.14 (SCL/A5), A1.32 (SCL/A5), R9.2
- net GPIO10: now also A1.20 (D5)
- net GPIO11: now also A1.21 (D6)
- net GPIO12: now also A1.22 (D7)
- net GPIO17: now also A1.28 (D13), J2.22; no longer J2.24
- net GPIO18: now also A1.27 (D12), J2.24; no longer J2.22
- net GPIO2: now also A1.13 (SDA/A4), A1.31 (SDA/A4), R8.2
- net GPIO3: now also A1.12 (A3)
- net GPIO33: now also A1.26 (D11)
- net GPIO34: now also A1.25 (D10)
- net GPIO35: now also A1.24 (D9)
- net GPIO36: now also A1.23 (D8)
- net GPIO4: now also A1.11 (A2)
- net GPIO5: now also A1.10 (A1)
- net GPIO6: now also A1.9 (A0)
- net GPIO7: now also A1.17 (D2)
- net GPIO8: now also A1.18 (D3)
- net GPIO9: now also A1.19 (D4)
- net U0RXD: now also A1.15 (D0/RX)
- net U0TXD: now also A1.16 (D1/TX)
- net VBUS: now also A1.8 (VIN), C1.1, IC1.2 (VIN_1), IC1.4 (VIN_2)
- net +5V: now reaches A1.5 (+5V)
- net +5V: now also C2.1, IC1.3 (VOUT)
Other:
- note added: "Arduino Pinout"
- note added: "B-Key-Female"
- note added: "BOOT Button"
- note added: "Pull-Up"
- note added: "RST Button"
- note added: "VBUS -> +5V"
- note removed: "B-Key"
- company: (none) -> LiberBoard
- title: (none) -> LiBo ArduinoBoard
- moved on the sheet: A1, C4, C5, C7, J1, L1, LED1, R2, R3, R4, R5, R6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

Commit message: first release
Parts:
- C4, C5, L1, R5, R6, U2: now not fitted
Connections:
- net GPIO10: now also A1.25 (D10); no longer A1.20 (D5)
- net GPIO11: now also A1.24 (D9); no longer A1.21 (D6)
- net GPIO12: now also A1.23 (D8); no longer A1.22 (D7)
- net GPIO17: now also A1.17 (D2); no longer A1.28 (D13)
- net GPIO18: now also A1.18 (D3); no longer A1.27 (D12)
- net GPIO33: now also A1.19 (D4); no longer A1.26 (D11)
- net GPIO34: now also A1.20 (D5); no longer A1.25 (D10)
- net GPIO35: now also A1.21 (D6); no longer A1.24 (D9)
- net GPIO36: now also A1.22 (D7); no longer A1.23 (D8)
- net GPIO45: now also LED1.3 (DI)
- net GPIO46: no longer LED1.3 (DI)
- net GPIO7: now also A1.28 (D13); no longer A1.17 (D2)
- net GPIO8: now also A1.27 (D12); no longer A1.18 (D3)
- net GPIO9: now also A1.26 (D11); no longer A1.19 (D4)
- net USB_D+: now also U1.4 (I/O2); no longer U1.1 (I/O1)
- net USB_D-: now also U1.1 (I/O1); no longer U1.4 (I/O2)
Other:
- note added: "DIT MOET EEN DIODE WORDEN"

Commit message: Add new STEP and WRL files for M.2 Arduino and ESP32S3 Boards
- Added M.2 Arduino Module Board STEP file (12633 KB)
- Added ESP32S3 M.2 Board STEP file (16645 KB)
- Added WRL file for unnamed ESP32S3 M.2 Board (2692 KB)
- Created lock file for ESP32S3 M.2 Board project
Parts:
- A1: value ~ -> (none)
